File: HW/PCB_TeensyLC/arduSynth.sch (KiCad schematic (older format))
At the start: 36 parts, among them J1 AudioJack3_Ground, J10 Conn_01x03_Male, J11 Screw_Terminal_01x02, J12 Conn_01x02_Male, J13 Conn_01x02_Male, J14 Screw_Terminal_01x02, J2 Conn_01x03_Male, J3 Conn_01x03_Male, J4 Conn_01x03_Male, J5 Conn_01x03_Male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

Commit message: updates for TeensyLC Version
Parts:
- added H1, H2, H3: MountingHole, MountingHole:MountingHole_3.2mm_M3_Pad, symbol Mechanical:MountingHole
- added J15: display_connector_91601-304LF, TeensySynth_Footprints:91601304LF, symbol SSD1306_display_connector:dispaly_connector_91601-304LF
- added J16, J17: Conn_01x03_Male, Connector_PinHeader_2.54mm:PinHeader_1x03_P2.54mm_Vertical, symbol Connector:Conn_01x03_Male
- added R5, R6: 4.7K, Resistor_THT:R_Axial_DIN0204_L3.6mm_D1.6mm_P2.54mm_Vertical, symbol Device:R_US
- J1: footprint test:FC68125 -> TeensySynth_Footprints:FC68125
- R1, R2, R3: footprint Resistors_THT:R_Axial_DIN0204_L3.6mm_D1.6mm_P2.54mm_Vertical -> Resistor_THT:R_Axial_DIN0204_L3.6mm_D1.6mm_P2.54mm_Vertical
- U1: footprint Teensy:Teensy_LC -> TeensySynth_Footprints:Teensy_LC; symbol teensy:Teensy-LC -> arduSynth-rescue:Teensy-LC-teensy
Connections:
- net +3V3: now also J15.3, R5.1, R6.1
- net +5V: now also U1.33 (Vin), J16.1 (Pin_1), J17.1 (Pin_1); no longer U1.15 (17_Vin)
- net GND: now also J15.1, J16.3 (Pin_3), J17.3 (Pin_3)
- net at C1.1, RV9.1: now also R4.2; no longer R4.1
- net AudioOut: now reaches U1.19 (26_A12/DAC)
- net AudioOut: now also R4.1; no longer R4.2
- net at J2.1 (Pin_1), J2.2 (Pin_2): now also U1.36 (24_A10); no longer U1.29 (22_A8_SCL1_PWM_Touch)
- net DataIn: now reaches U1.2 (0_RX1_MOSI1_Touch)
- net DataIn: now also J16.2 (Pin_2)
- net DataOut: now reaches U1.3 (1_TX1_MISO1_Touch)
- net DataOut: now also J17.2 (Pin_2)
- net SDA: now reaches U1.30 (23_A9_SDA1_PWM_Touch)
- net SDA: now also J15.7, R6.2
- new net SCL: J15.5, R5.2, U1.29 (22_A8_SCL1_PWM_Touch)
Other:
- moved on the sheet: C1, J1, J10, J11, J12, J13, J14, R4, RV9

Commit message: some final PCB updates for Teensynth V1.0
Parts:
- removed J11, J14: Screw_Terminal_01x02, TerminalBlock:TerminalBlock_bornier-2_P5.08mm, symbol Connector:Screw_Terminal_01x02
- added J11: Screw_Terminal_01x03, TerminalBlock:TerminalBlock_bornier-3_P5.08mm, symbol Connector:Screw_Terminal_01x03
Connections:
- net +3V3: now also J11.1 (Pin_1)
- net GND: now also J11.3 (Pin_3)
- net at J10.1 (Pin_1), J10.2 (Pin_2), J10.3 (Pin_3): now also J11.2 (Pin_2)
Changed lines of the file:
@@
 Connection ~ 8950 5950
-$Comp
-L Connector:Screw_Terminal_01x02 J14
-U 1 1 61228DB8
-P 1500 1100
-F 0 "J14" V 1800 1100 50  0000 R CNN
-F 1 "Screw_Terminal_01x02" V 1700 1450 50  0000 R CNN
-F 2 "TerminalBlock:TerminalBlock_bornier-2_P5.08mm" H 1500 1100 50  0001 C CNN
-F 3 "~" H 1500 1100 50  0001 C CNN
-	1    1500 1100
-	0    -1   -1   0
-$EndComp
-$Comp
-L Connector:Screw_Terminal_01x02 J11
-U 1 1 612296C7
-P 3250 1050
-F 0 "J11" V 3500 1100 50  0000 R CNN
-F 1 "Screw_Terminal_01x02" V 3400 1400 50  0000 R CNN
-F 2 "TerminalBlock:TerminalBlock_bornier-2_P5.08mm" H 3250 1050 50  0001 C CNN
-F 3 "~" H 3250 1050 50  0001 C CNN
-	1    3250 1050
-	0    -1   -1   0
-$EndComp
 $Comp
 L Connector:Conn_01x02_Male J12
@@
 Connection ~ 3350 5650
 $Comp
-L power:GND #PWR0130
-U 1 1 612467D9
-P 1600 1500
-F 0 "#PWR0130" H 1600 1250 50  0001 C CNN
-F 1 "GND" H 1605 1327 50  0000 C CNN
-F 2 "" H 1600 1500 50  0001 C CNN
-F 3 "" H 1600 1500 50  0001 C CNN
-	1    1600 1500
-	1    0    0    -1
-$EndComp
-Wire Wire Line
-	1600 1300 1600 1500
-$Comp
 L power:GND #PWR0131
 U 1 1 6124BDD7
@@
 Wire Wire Line
 	5250 4250 5150 4250
-$Comp
-L power:+5V #PWR0132
-U 1 1 6172BB98
-P 1500 1300
-F 0 "#PWR0132" H 1500 1150 50  0001 C CNN
-F 1 "+5V" H 1515 1473 50  0000 C CNN
-F 2 "" H 1500 1300 50  0001 C CNN
-F 3 "" H 1500 1300 50  0001 C CNN
-	1    1500 1300
-	-1   0    0    1
-$EndComp
 $Comp
 L power:+5V #PWR0133
@@
 	1    0    0    -1
 $EndComp
+$Comp
+L Connector:Screw_Terminal_01x03 J11
+U 1 1 6177C5E9
+P 3250 1050
+F 0 "J11" V 3214 862 50  0000 R CNN
+F 1 "Screw_Terminal_01x03" V 3123 862 50  0000 R CNN
+F 2 "TerminalBlock:TerminalBlock_bornier-3_P5.08mm" H 3250 1050 50  0001 C CNN
+F 3 "~" H 3250 1050 50  0001 C CNN
+	1    3250 1050
+	0    -1   -1   0
+$EndComp
+$Comp
+L power:+3.3V #PWR03
+U 1 1 6178DD15
+P 2850 1050
+F 0 "#PWR03" H 2850 900 50  0001 C CNN
+F 1 "+3.3V" V 2850 1300 50  0000 C CNN
+F 2 "" H 2850 1050 50  0001 C CNN
+F 3 "" H 2850 1050 50  0001 C CNN
+	1    2850 1050
+	1    0    0    -1
+$EndComp
+Wire Wire Line
+	3150 1250 2850 1250
+Wire Wire Line
+	2850 1250 2850 1050
 $EndSCHEMATC
